File: MainBoard/v4.2/linearSensor.brd (EAGLE design)
At the start: 40.6 x 30.7 mm, 19 parts, among them CON1 SPI, X1 FH12-08S-1SH, X3 16MHz, X4 MINI-USB

Commit message: Add new corrected version
Parts:
- moved C12 6.35 mm to (13.0, 1.91)
- moved C7 3.27 mm to (13.7, 27.9), turned to 90 degrees
- moved R24 1.80 mm to (14.0, 21.6)
- moved C10 1.27 mm to (16.5, 27.9), turned to 90 degrees
- moved C11 1.27 mm to (2.86, 8.57)
- moved R31 1.27 mm to (16.5, 21.6)
Connections:
- net D+USB renamed D_USB+
- net D-USB renamed D_USB-
Routing:
- net GND: track 0.00 -> 180.7 mm, vias 0 -> 4
- net +5V/1: track 0.00 -> 151.7 mm, vias 0 -> 8
- net MISO: track 0.00 -> 75.0 mm, vias 0 -> 1
- net SCK: track 0.00 -> 67.3 mm, vias 0 -> 3
- net D7*: track 0.00 -> 56.8 mm, vias 0 -> 2
- net RESET: track 0.00 -> 55.5 mm, vias 0 -> 1
- net A2: track 0.00 -> 49.8 mm, vias 0 -> 2
- net RD+: track 0.00 -> 46.3 mm
- net RD-: track 0.00 -> 46.0 mm
- net MOSI: track 0.00 -> 43.7 mm, vias 0 -> 3
- net A4: track 0.00 -> 34.1 mm, vias 0 -> 2
- net D13*: track 0.00 -> 33.4 mm, vias 0 -> 2
- net A3: track 0.00 -> 31.0 mm, vias 0 -> 2
- net A1: track 0.00 -> 29.4 mm, vias 0 -> 1
- net D6*: track 0.00 -> 29.4 mm, vias 0 -> 2
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