File: simple-spectro/simple_spectro.brd (EAGLE design)
At the start: 70.5 x 40.5 mm, 56 parts, among them CN2 JSTPH, U1 MCP73831T-2ACI/OT, X2 16MHz, X4 MINI-USB

Commit message: starting disposition of components in simple spectro
Parts:
- removed C11: 100nF, rcl:C1206
- removed CN1: (no value), microbuilder:USBA_PCB
- removed CN2: JSTPH, microbuilder:JSTPH2
- removed LCD: (no value), lpatiny:1X16
- removed R6: 2K, microbuilder:0805
- removed RK6: 10k, resistor:M0805
- removed SJ1: (no value), jumper:SJ
- removed SJ2: (no value), microbuilder:SOLDERJUMPER_ARROW_NOPASTE
- added C4: 100nF, dp_devices:C805
- added CON2: JACK_DC_BARREL, lpatiny:DC_BARREL
- added CU7, CU8: 10u, rcl:C0805
- added D1, D3, D5, D6: 1N581D1206, lpatiny:LED-1206
- added IC1: MCP1703DB, linear:SOT223
- added J2: RJ12RIGHTANGLE-I2C, lpatiny:RJ12-RIGHTANGLE-I2C
- added PAD1, PAD2: (no value), wirepad:SMD1,27-2,54
- added Q1: DMP1045U, dp_devices:SOT-23
- added U$11: LCD-HD447804-HOLES16X2-4-HOLES, HD44780LCD:LCD-16X2-4HOLES
- R3: value 1k -> 100k; device rcl:R0805 -> microbuilder:0805
- RK1: value 10k -> 3.9k
- moved CU5 150.1 mm to (-6.35, -120.7), flipped to the top, turned to 0 degrees
- moved CU6 149.6 mm to (0.00, -120.7), flipped to the top, turned to 0 degrees
- moved LDO 146.8 mm to (-6.35, -110.5), flipped to the top
- moved U1 90.8 mm to (59.1, 25.6)
- moved U$9 89.4 mm to (58.8, 12.2), turned to 270 degrees
- moved 220 71.7 mm to (45.4, 65.3), turned to 0 degrees
- moved CX1 69.6 mm to (49.1, 61.0), turned to 270 degrees
- moved RXT 60.3 mm to (47.0, 56.4), turned to 90 degrees
- moved C2 59.0 mm to (24.9, 21.3)
- moved C3 59.0 mm to (30.6, 21.3)
- moved R1 59.0 mm to (11.2, 14.7)
- moved R4 59.0 mm to (16.9, 14.7)
- moved R5 59.0 mm to (22.6, 14.7)
- moved LED1 59.0 mm to (11.4, 10.2)
- moved LED2 59.0 mm to (15.6, 10.2)
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Connections:
- removed net VDD1: C2.1, CN1.VCC, LED1.A, U1.4
- new net I2C-5V: D1.A, J2.+5V
- new net N$15: C2.1, D4.C, D5.A, D6.C, LED1.A, Q1.1, R3.2, U1.4
- new net VCC: 32U4.13, CU8.1, IC1.3
- new net VDD: CU7.1, D5.C, IC1.1, Q1.2
- net +12V: now also D3.A, J2.+12V
- net +5V/1: now also D1.C, D6.A, U$11.2; no longer 32U4.2, D4.C, LCD.2, RK1.1, RK6.2
- net A6: now also U$11.14; no longer LCD.14
- net D10*: now also U$11.4; no longer LCD.4
- net D12*: now also U$11.13; no longer LCD.13
- net D13*: now also RK1.1
- net D6*: now also U$11.12; no longer LCD.12
- net D8*: now also U$11.11; no longer LCD.11
- net D9*: now also U$11.6; no longer LCD.6
- net GND: now also C4.2, CON2.P$2, CU7.2, CU8.2, IC1.2, J2.GND1, J2.GND2, PAD2.1, R3.1, U$11.1, U$11.16, U$11.5; no longer C11.2, CN1.GND, CN2.1, LCD.1, LCD.16, LCD.5, R3.2, R6.2, SJ1.1
- net N$11: now also U$11.15; no longer LCD.15
- net N$2: now also C4.1, U$11.3; no longer LCD.3, R3.1
- net N$6: no longer SJ2.2
- net N$8: now also D3.C; no longer R6.1, SJ2.1
- net RESET: no longer 32U4.13, C11.1, RK6.1, SJ1.2
- net SCL: now also J2.SCL
- net SDA: now also J2.SDA
- net VBAT1: now also PAD1.1, Q1.3; no longer CN2.2
- net VUSB: now also 32U4.2
Routing:
- net +5V/1: track 214.9 -> 0.00 mm, vias 6 -> 0
- net GND: track 80.8 -> 0.00 mm, vias 17 -> 0
- net D7*: track 53.8 -> 0.00 mm, vias 3 -> 0
- net TX: track 48.4 -> 0.00 mm, vias 3 -> 0
- net VUSB: track 45.8 -> 0.00 mm, vias 2 -> 0
- net SCK: track 45.6 -> 0.00 mm, vias 3 -> 0
- net RESET: track 39.0 -> 0.00 mm, vias 1 -> 0
- net RX: track 35.7 -> 0.00 mm, vias 2 -> 0
- net MISO: track 28.4 -> 0.00 mm, vias 2 -> 0
- net MOSI: track 27.1 -> 0.00 mm, vias 1 -> 0
- net N$42: track 19.8 -> 0.00 mm
- net XTAL1: track 18.4 -> 0.00 mm
- net A6: track 16.9 -> 0.00 mm
- net D12*: track 15.9 -> 0.00 mm
- net D6*: track 14.0 -> 0.00 mm
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- removed copper zone on layer 16, net GND
Other:
- board size 70.5 x 40.5 mm -> 99.1 x 73.7 mm

Commit message: Update simple spectro
Parts:
- removed 5V1, GND: (no value), Headerlibrary:1X01
- removed CU5, CU6: 10uF, rcl:C1206
- removed LDO: NCP1117LPST50T3G, lpatiny:SOT223
- added L1: UV, led:LED3MM
- added Q2: DMP1045U, dp_devices:SOT-23
- added R6, R8: 470, microbuilder:0805
- added R9: 1k, rcl:R0805
- moved CU7 172.5 mm to (64.1, 55.9), turned to 90 degrees
- moved CU8 130.2 mm to (35.6, 23.5)
- moved RL4 121.0 mm to (57.4, 42.0)
- moved R7 116.0 mm to (48.1, 21.6)
- moved BKLD1 116.0 mm to (49.0, 27.6)
- moved C4 116.0 mm to (48.3, 15.9)
- moved IC1 116.0 mm to (50.2, 8.89)
- moved RL2 116.0 mm to (48.1, 35.7)
- moved RL3 116.0 mm to (53.4, 35.7)
- moved LED1 66.5 mm to (59.7, 55.9)
- moved PAD1 11.7 mm to (73.0, 69.8)
- moved PAD2 11.7 mm to (69.2, 69.8)
- moved R4 11.4 mm to (16.9, 26.1)
- moved RK7 8.66 mm to (12.5, 62.6), turned to 270 degrees
- moved Q1 7.73 mm to (62.9, 61.6)
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Connections:
- removed net BLUE: RL2.2
- removed net GREEN: RL3.2
- removed net RED: RL4.1
- new net N$17: D4.C, D6.C, Q2.3
- new net N$18: Q2.1, R6.1, R8.2
- new net N$19: L1.A, R9.2
- net +12V: no longer CU6.1, LDO.3
- net +5V/1: now also R8.1; no longer 220.1, 5V1.1, CU5.1, LDO.2, LDO.4, U$11.2
- net A0: now also RL2.2
- net A1: now also RL4.1
- net A2: now also RL3.2
- net A3: now also R9.1
- net D11*: now also 220.1
- net GND: now also L1.K; no longer CU5.2, CU6.2, GND.1, LDO.1
- net MOSI: now also U$11.2
- net N$15: now also Q2.2; no longer D4.C, D6.C
- net VCC: now also R6.2

Commit message: Start routing
Parts:
- removed BKLD: RED, adafruit:CHIP-LED0805
- removed C1: 100nF, rcl:C1206
- removed CU3, CU9: 10uF, rcl:C1206
- removed D2, D3: 1N581D1206, lpatiny:LED-1206
- removed PAD1, PAD2: (no value), wirepad:SMD1,27-2,54
- removed R2: 1k, rcl:R0805
- added CU1: 100nF, rcl:C0805
- added D7, D8: 1N581D1206, lpatiny:LED-1206
- added RK3: 10k, resistor:M0805
- added U$12: CONN2, lpatiny:JST-2-XH
- added U$7: TSL237, lpatiny:TSL237
- X2: value 16MHz -> 8MHz
- moved RK2 82.5 mm to (88.9, 15.9), flipped to the bottom
- moved R8 77.4 mm to (74.3, 45.7), flipped to the bottom
- moved Q2 75.5 mm to (71.1, 59.7), flipped to the bottom
- moved R6 70.8 mm to (67.9, 55.2), flipped to the bottom, turned to 270 degrees
- moved R1 68.4 mm to (59.1, 63.5), flipped to the bottom, turned to 180 degrees
- moved R5 66.6 mm to (69.2, 62.2), flipped to the bottom
- moved C2 65.7 mm to (69.2, 69.8), flipped to the bottom
- moved LED2 63.6 mm to (54.0, 61.0), flipped to the bottom, turned to 270 degrees
- moved RE2 62.9 mm to (66.7, 12.7), flipped to the bottom
- moved RE1 59.3 mm to (66.7, 15.2), flipped to the bottom
- moved C3 56.3 mm to (64.8, 66.0), flipped to the bottom, turned to 270 degrees
- moved C4 54.9 mm to (17.8, 61.6), flipped to the bottom, turned to 180 degrees
- moved R4 54.7 mm to (59.1, 61.0), flipped to the bottom, turned to 180 degrees
- moved U1 41.7 mm to (69.2, 66.0), flipped to the bottom, turned to 90 degrees
- moved IC1 40.6 mm to (57.1, 48.9), flipped to the bottom
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Connections:
- removed net +12V: D3.A, J2.+12V
- removed net +5V/1: 32U4.14, 32U4.24, 32U4.34, 32U4.44, C1.1, C12.2, CU3.1, D1.C, D2.C, D6.A, R13.1, R8.1, RE1.1, RE2.1, RK2.2
- removed net I2C-5V: D1.A, J2.+5V
- removed net N$17: D4.C, D6.C, Q2.3
- removed net N$3: BKLD.A, R2.2
- removed net N$8: D3.C
- new net EXT-VCC: D1.A
- new net HIGH-VCC: D1.C, D6.C, Q2.3, R8.1
- new net I2C+12V: D6.A, J2.+12V
- new net I2C+5V: D7.A, J2.+5V
- net A0: no longer RL2.2
- net A1: now also RL2.2; no longer RL4.1
- net A2: now also RL4.1; no longer RL3.2
- net A3: now also RL3.2; no longer R9.1
- net A4: now also R9.1
- net A5: now also R7.1
- net A6: now also U$11.4; no longer U$11.14
- net D10*: now also U$11.14; no longer U$11.4
- net D12*: now also U$11.6; no longer U$11.13
- net D13*: no longer R2.1, R7.1
- net D5*: now also U$7.OUT
- net D6*: now also U$11.11; no longer U$11.12
- net D8*: now also U$11.12; no longer U$11.11
- net D9*: now also U$11.13; no longer U$11.6
- net GND: now also CU1.2, U$12.1, U$7.GND; no longer BKLD.C, C1.2, CU3.2, CU9.1, PAD2.1
- net ISP+5V: now also D8.A; no longer D2.A
- net N$15: now also D4.C, D7.C, D8.C
- net RESET: now also 32U4.13, RK3.1
- net VBAT1: now also U$12.2; no longer PAD1.1
- net VCC: now also 32U4.14, 32U4.24, 32U4.34, 32U4.44, C12.2, CU1.1, R13.1, RE1.1, RE2.1, RK2.2, RK3.2, U$7.VDD; no longer 32U4.13
- net VUSB: no longer CU9.2
Routing:
- net ISP+5V: track 0.00 -> 137.6 mm, vias 0 -> 2
- net GND: track 0.00 -> 125.4 mm
- net RX: track 0.00 -> 90.5 mm, vias 0 -> 1
- net TX: track 0.00 -> 88.7 mm, vias 0 -> 1
- net D7*: track 0.00 -> 84.5 mm, vias 0 -> 1
- net VUSB: track 0.00 -> 72.1 mm, vias 0 -> 2
- net SCL: track 0.00 -> 65.9 mm, vias 0 -> 1
- net SDA: track 0.00 -> 63.6 mm, vias 0 -> 1
- net D5*: track 0.00 -> 61.4 mm, vias 0 -> 2
- net USBC_P: track 0.00 -> 57.8 mm, vias 0 -> 2
- net USBC_N: track 0.00 -> 53.9 mm, vias 0 -> 2
- net VCC: track 0.00 -> 53.0 mm
- net A1: track 0.00 -> 52.6 mm
- net A2: track 0.00 -> 49.3 mm
- net A3: track 0.00 -> 46.0 mm
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Other:
- outline, holes or cut-outs redrawn
- board text removed: "C:/Users/G/Pictures/logo_epfl.bmp"
- board text removed: "Screen v0.1"

Commit message: work in progress
Parts:
- removed CON2: JACK_DC_BARREL, lpatiny:DC_BARREL
- removed D1: 1N581D1206, lpatiny:LED-1206
- removed Q2: DMP1045U, dp_devices:SOT-23
- removed R6, R8: 470, microbuilder:0805
- added IC2: MCP1703-50, linear:SOT223
- IC1: value MCP1703DB -> MCP1703-33
- moved D4 28.6 mm to (73.7, 62.2), turned to 90 degrees
- moved R3 16.2 mm to (73.7, 69.2), turned to 270 degrees
- moved X4 14.0 mm to (87.6, 43.2)
- moved D6 3.24 mm to (76.8, 52.7), turned to 270 degrees
Connections:
- removed net EXT-VCC: D1.A
- removed net N$18: Q2.1, R6.1, R8.2
- net GND: now also IC2.2; no longer CON2.P$2
- net HIGH-VCC: now also IC2.1; no longer D1.C, Q2.3, R8.1
- net N$15: now also IC2.3; no longer Q2.2
- net VCC: no longer R6.2
Routing:
- net N$15: track 11.1 -> 44.7 mm
- net USBC_P: track 57.8 -> 73.1 mm
- net USBC_N: track 53.9 -> 69.0 mm, vias 2 -> 3
- net VUSB: track 72.1 -> 87.0 mm
- net I2C+12V: track 0.00 -> 7.63 mm
- net I2C+5V: track 0.00 -> 6.73 mm
- net HIGH-VCC: track 0.00 -> 3.73 mm

Commit message: removed useless D6 schottky
Parts:
- removed D6: 1N581D1206, lpatiny:LED-1206
Connections:
- removed net HIGH-VCC: D6.C, IC2.1
- net I2C+12V: now also IC2.1; no longer D6.A
Routing:
- net HIGH-VCC: track 3.73 -> 0.00 mm
- net I2C+12V: track 7.63 -> 9.36 mm
Changed lines of the file:
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@@
 <?xml version="1.0" encoding="utf-8"?>
 <!DOCTYPE eagle SYSTEM "eagle.dtd">
-<eagle version="7.7.0">
+<eagle version="7.5.0">
 <drawing>
 <settings>
@@
 <element name="D5" library="lpatiny" package="LED-1206" value="1N581D1206" x="65.405" y="40.005" rot="MR0"/>
 <element name="D4" library="lpatiny" package="LED-1206" value="1N581D1206" x="73.66" y="62.23" rot="MR90"/>
-<element name="D6" library="lpatiny" package="LED-1206" value="1N581D1206" x="76.835" y="52.705" rot="MR270"/>
 <element name="R9" library="rcl" package="R0805" value="1k" x="32.385" y="27.94" rot="MR180"/>
 <element name="L1" library="led" package="LED3MM" value="UV" x="37.465" y="27.94"/>
@@
 <signal name="I2C+12V" class="1">
 <contactref element="J2" pad="+12V"/>
-<contactref element="D6" pad="A"/>
-<wire x1="76.835" y1="54.205" x2="76.835" y2="55.88" width="0.4064" layer="16"/>
 <wire x1="76.835" y1="55.88" x2="82.79" y2="55.88" width="0.4064" layer="16"/>
-</signal>
-<signal name="HIGH-VCC">
-<contactref element="D6" pad="C"/>
 <contactref element="IC2" pad="1"/>
 <wire x1="73.4314" y1="50.8762" x2="76.835" y2="50.8762" width="0.4064" layer="16"/>
-<wire x1="76.835" y1="50.8762" x2="76.835" y2="51.205" width="0.4064" layer="16"/>
+<wire x1="76.835" y1="50.8762" x2="76.835" y2="55.88" width="0" layer="19" extent="16-16"/>
 </signal>
 </signals>

Commit message: work in progress
Parts:
- removed RE1, RE2: 5k, rcl:R0805
- removed RK2: 10k, resistor:M0805
- added CON_ISP1: SPI, lpatiny:TINYISP
- added L2: UV, led:LED3MM
- added R2: 1k, rcl:R0805
- L1: device led:LED3MM -> SparkFun:LED5MM
- RK3: value 10k -> 100k
- moved RUSB2 50.9 mm to (83.8, 41.3), turned to 180 degrees
- moved RUSB1 48.2 mm to (83.8, 45.7), turned to 180 degrees
- moved R9 19.1 mm to (51.4, 26.0), turned to 0 degrees
- moved CU7 14.8 mm to (67.9, 41.9), turned to 0 degrees
- moved D4 10.2 mm to (83.8, 62.2)
- moved Q1 8.35 mm to (73.7, 45.7)
- moved D5 8.28 mm to (73.7, 40.6)
- moved LED2 7.67 mm to (61.0, 64.1)
- moved CU1 7.65 mm to (63.5, 39.4)
- moved CU8 7.65 mm to (63.5, 41.9)
- moved IC1 7.65 mm to (64.8, 48.3)
- moved LDPW5 7.65 mm to (64.8, 35.6)
- moved R13 7.65 mm to (62.2, 35.6)
- moved LED1 7.43 mm to (61.0, 61.0)
- moved R1 6.84 mm to (65.4, 61.0)
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Connections:
- new net N$8: L2.A, R2.2
- net A0: now also RL2.2
- net A1: now also RL4.1; no longer RL2.2
- net A2: now also RL3.2; no longer RL4.1
- net A3: now also R2.1; no longer RL3.2
- net D7*: no longer RK2.1
- net GND: now also CON_ISP1.GND, L2.K
- net ISP+5V: now also CON_ISP1.VCC
- net MISO: now also CON_ISP1.MISO
- net MOSI: now also CON_ISP1.MOSI
- net RESET: now also CON_ISP1.RESET
- net RX: no longer RE2.2
- net SCK: now also CON_ISP1.SCK
- net TX: no longer RE1.2
- net VCC: no longer RE1.1, RE2.1, RK2.2
Routing:
- net USBC_P: track 73.1 -> 7.67 mm, vias 2 -> 0
- net MOSI: track 12.0 -> 75.6 mm, vias 2 -> 3
- net USB_P: track 6.70 -> 69.0 mm, vias 0 -> 2
- net USBC_N: track 69.0 -> 7.50 mm, vias 3 -> 0
- net USB_N: track 8.81 -> 69.9 mm, vias 0 -> 2
- net A0: track 0.00 -> 53.4 mm
- net SCK: track 16.6 -> 68.2 mm
- net MISO: track 12.4 -> 58.2 mm, vias 0 -> 2
- net VBAT1: track 13.4 -> 57.7 mm
- net VUSB: track 87.0 -> 127.3 mm
- net RESET: track 23.4 -> 59.9 mm, vias 0 -> 1
- net VCC: track 53.0 -> 88.8 mm, vias 0 -> 1
- net N$15: track 44.7 -> 69.7 mm
- net GND: track 125.4 -> 143.3 mm, vias 0 -> 9
- net ISP+5V: track 137.6 -> 155.3 mm
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- added copper zone on layer 1, net GND

Commit message: first version of simple spectro
Connections:
- removed net GND1: U$9.GND
- net GND: now also U$9.GND
Changed lines of the file:
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@@
 <wire x1="27.305" y1="40.7162" x2="27.0764" y2="40.9448" width="0.4064" layer="16"/>
 <via x="27.0764" y="40.9448" extent="1-16" drill="0.3048" shape="square"/>
-<wire x1="74.93" y1="62.23" x2="77.47" y2="50.8762" width="0" layer="19" extent="16-16"/>
-<wire x1="37.63" y1="45" x2="42.63" y2="47.6" width="0" layer="19" extent="16-16"/>
 <via x="77.47" y="48.895" extent="1-16" drill="0.3048" shape="square"/>
-<wire x1="77.47" y1="48.895" x2="78.105" y2="48.895" width="0" layer="19" extent="1-16"/>
-<wire x1="78.105" y1="48.895" x2="88.265" y2="41.58" width="0" layer="19" extent="1-16"/>
+<contactref element="U$9" pad="GND"/>
+<wire x1="42.63" y1="47.6" x2="37.63" y2="45" width="0" layer="19" extent="16-16"/>
 </signal>
 <signal name="SCK">
@@
 <contactref element="LED2" pad="A"/>
 <wire x1="64.455" y1="63.5" x2="62.01" y2="64.135" width="0.4064" layer="16"/>
-</signal>
-<signal name="GND1" class="1">
-<contactref element="U$9" pad="GND"/>
 </signal>
 <signal name="N$9">
@@
 <wire x1="31.75" y1="40.64" x2="32.385" y2="40.64" width="0.4064" layer="1"/>
 <wire x1="32.385" y1="40.64" x2="32.385" y2="33.655" width="0.4064" layer="1"/>
-<wire x1="5.715" y1="72.39" x2="7.62" y2="72.39" width="0" layer="19" extent="1-16"/>
 <wire x1="7.62" y1="72.39" x2="83.185" y2="72.39" width="0.4064" layer="16"/>
 <wire x1="83.185" y1="72.39" x2="83.185" y2="70.715" width="0.4064" layer="16"/>

Commit message: Update
Parts:
- removed C3: 10µF, microbuilder:0805
- removed D5: 1N581D1206, lpatiny:LED-1206
- removed L1: UV, SparkFun:LED5MM
- removed L2: UV, led:LED3MM
- removed LED1: RED, microbuilder:CHIPLED_0805
- removed LED2: GREEN, microbuilder:CHIPLED_0805
- removed Q1: DMP1045U, dp_devices:SOT-23
- removed R1, R4: 470, microbuilder:0805
- removed R2, R9: 1k, rcl:R0805
- removed R3: 100k, microbuilder:0805
- removed R5: 10K\, microbuilder:0805
- removed RL2, RL4: 150, rcl:R0805
- removed RL3: 100, rcl:R0805
- removed U$12: CONN2, lpatiny:JST-2-XH
- removed U$7: TSL237, lpatiny:TSL237
- removed U$9: RGB-COMMON-CATHODE, lpatiny:LED-TRICOLOR-THROUGHHOLE
- removed U1: MCP73831T-2ACI/OT, microbuilder:SOT23-5
- IC1: value MCP1703-33 -> MCP1703-50
Connections:
- removed net N$10: RL3.1, U$9.BLU
- removed net N$13: RL2.1, U$9.RED
- removed net N$15: C2.1, D4.C, D5.A, D7.C, D8.C, IC2.3, LED1.A, Q1.1, R3.2, U1.4
- removed net N$3: L1.A, R9.2
- removed net N$4: LED1.C, R1.1
- removed net N$5: R1.2, R4.2, U1.1
- removed net N$6: R5.1, U1.5
- removed net N$7: LED2.A, R4.1
- removed net N$8: L2.A, R2.2
- removed net N$9: RL4.2, U$9.GRN
- removed net VBAT1: C3.1, Q1.3, U$12.2, U1.3
- new net N$19: C2.1, D4.C, D7.C, D8.C, IC2.3
- net A0: no longer RL2.2
- net A1: no longer RL4.1
- net A2: no longer RL3.2
- net A3: no longer R2.1
- net A4: no longer R9.1
- net D5*: no longer U$7.OUT
- net GND: no longer C3.2, L1.K, L2.K, LED2.C, R3.1, R5.2, U$12.1, U$7.GND, U$9.GND, U1.2
- net VCC: no longer U$7.VDD
- net VDD: no longer D5.C, Q1.2
Routing:
- net N$15: track 69.7 -> 0.00 mm
- net VBAT1: track 57.7 -> 0.00 mm
- net N$19: track 0.00 -> 52.8 mm
- net GND: track 143.3 -> 117.6 mm
- net N$10: track 15.2 -> 0.00 mm
- net N$5: track 14.6 -> 0.00 mm
- net N$9: track 11.2 -> 0.00 mm
- net N$3: track 7.30 -> 0.00 mm
- net N$8: track 6.67 -> 0.00 mm
- net N$13: track 5.83 -> 0.00 mm
- net A3: track 47.3 -> 42.2 mm
- net VDD: track 13.4 -> 8.88 mm
- net A4: track 42.0 -> 37.9 mm
- net N$6: track 3.21 -> 0.00 mm
- net A0: track 53.4 -> 50.3 mm
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