File: simple-spectro/simple-spectro.sch (EAGLE design)
At the start: 34 parts, among them IC1 MCP1703-50, IC2 MCP1703-50, J2 RJ12RIGHTANGLE-I2C, X2 8MHz, X4 MINI-USB

Commit message: Close to final
Parts:
- added C3: 10µF, microbuilder:CAP_CERAMIC0805
- added D5: 1N581D1206, lpatiny:1N581D1206
- added L1: UV, SparkFun:LED5MM
- added L2: UV, led:LED3MM
- added LED1: RED, microbuilder:LED0805
- added LED2: GREEN, microbuilder:LED0805
- added Q1: DMP1045U, dp_devices:TRANSISTOR_FET_TSM2301CX
- added R1, R4: 470, microbuilder:RESISTOR0805
- added R2, R9: 1k, rcl:R-EU_R0805
- added R3: 100k, microbuilder:RESISTOR0805
- added R5: 10K\, microbuilder:RESISTOR0805
- added RL2, RL4: 150, rcl:R-EU_R0805
- added RL3: 100, rcl:R-EU_R0805
- added U$12: CONN2, lpatiny:CONN2
- added U$7: TSL237, lpatiny:TSL237
- added U$9: RGB-COMMON-CATHODE, lpatiny:RGB-COMMON-CATHODE
- added U1: MCP73831T, microbuilder:MCP73831/2
- IC1: value MCP1703-50 -> MCP1703-33
Connections:
- removed net N$19: C2.P$1, D4.C, D7.C, D8.C, IC2.VO
- new net N$10: RL3.1, U$9.CBLUE
- new net N$13: RL2.1, U$9.CRED
- new net N$15: C2.P$1, D4.C, D5.A, D7.C, D8.C, IC2.VO, LED1.A, Q1.G, R3.2, U1.VDD
- new net N$3: L1.A, R9.2
- new net N$4: LED1.C, R1.1
- new net N$5: R1.2, R4.2, U1.STAT
- new net N$6: R5.1, U1.PROG
- new net N$7: LED2.A, R4.1
- new net N$8: L2.A, R2.2
- new net N$9: RL4.2, U$9.CGREEN
- new net VBAT1: C3.P$1, Q1.D, U$12.2, U1.VBAT
- net A0: now also RL2.2
- net A1: now also RL4.1
- net A2: now also RL3.2
- net A3: now also R2.1
- net A4: now also R9.1
- net D5*: now also U$7.OUT
- net GND: now also C3.P$2, L1.C, L2.C, LED2.C, R3.1, R5.2, U$12.1, U$7.GND, U$9.A2, U1.VSS
- net VCC: now also U$7.VDD
- net VDD: now also D5.C, Q1.S
Other:
- note added: "1.0K = 1000mA"
- note added: "10K = 100mA"
- note added: "2.0K = 500mA"
- note added: "3.3V LDO"
- note added: "5.0K = 200mA"
- note added: "Load sharing: http://blog.zakkemble.co.uk/a-lithium-battery-charger-with-load-sharing/"
- note added: "MAX 6V !"
- note added: "Over voltage protection * Consumption ? * Check resistance"
- note removed: "5.0V LDO"
