File: simple-spectro/simple-spectro.brd (EAGLE design)
At the start: 99.1 x 73.7 mm, 34 parts, among them IC1 MCP1703-50, IC2 MCP1703-50, J2 RJ12RIGHTANGLE-I2C, X2 8MHz, X4 MINI-USB

Commit message: Close to final
Parts:
- added C3: 10µF, microbuilder:0805
- added D5: 1N581D1206, lpatiny:LED-1206
- added L1: UV, SparkFun:LED5MM
- added L2: UV, led:LED3MM
- added LED1: RED, microbuilder:CHIPLED_0805
- added LED2: GREEN, microbuilder:CHIPLED_0805
- added Q1: DMP1045U, dp_devices:SOT-23
- added R1, R4: 470, microbuilder:0805
- added R2, R9: 1k, rcl:R0805
- added R3: 100k, microbuilder:0805
- added R5: 10K\, microbuilder:0805
- added RL2, RL4: 150, rcl:R0805
- added RL3: 100, rcl:R0805
- added U$12: CONN2, lpatiny:JST-2-XH
- added U$7: TSL237, lpatiny:TSL237
- added U$9: RGB-COMMON-CATHODE, lpatiny:LED-TRICOLOR-THROUGHHOLE
- added U1: MCP73831T, microbuilder:SOT23-5
- IC1: value MCP1703-50 -> MCP1703-33
- moved D4 0.63 mm to (83.2, 62.2)
Connections:
- removed net N$19: C2.1, D4.C, D7.C, D8.C, IC2.3
- new net N$10: RL3.1, U$9.BLU
- new net N$13: RL2.1, U$9.RED
- new net N$15: C2.1, D4.C, D5.A, D7.C, D8.C, IC2.3, LED1.A, Q1.1, R3.2, U1.4
- new net N$3: L1.A, R9.2
- new net N$4: LED1.C, R1.1
- new net N$5: R1.2, R4.2, U1.1
- new net N$6: R5.1, U1.5
- new net N$7: LED2.A, R4.1
- new net N$8: L2.A, R2.2
- new net N$9: RL4.2, U$9.GRN
- new net VBAT1: C3.1, Q1.3, U$12.2, U1.3
- net A0: now also RL2.2
- net A1: now also RL4.1
- net A2: now also RL3.2
- net A3: now also R2.1
- net A4: now also R9.1
- net D5*: now also U$7.OUT
- net GND: now also C3.2, L1.K, L2.K, LED2.C, R3.1, R5.2, U$12.1, U$7.GND, U$9.GND, U1.2
- net VCC: now also U$7.VDD
- net VDD: now also D5.C, Q1.2
Routing:
- net N$15: track 0.00 -> 69.1 mm
- net VBAT1: track 0.00 -> 57.7 mm
- net N$19: track 52.8 -> 0.00 mm
- net GND: track 117.6 -> 143.3 mm
- net N$5: track 0.00 -> 15.2 mm
- net N$10: track 0.00 -> 15.2 mm
- net N$9: track 0.00 -> 11.2 mm
- net N$3: track 0.00 -> 7.30 mm
- net N$8: track 0.00 -> 6.67 mm
- net N$13: track 0.00 -> 5.83 mm
- net A3: track 42.2 -> 47.3 mm
- net VDD: track 8.88 -> 13.4 mm
- net A4: track 37.9 -> 42.0 mm
- net N$6: track 0.00 -> 3.21 mm
- net A0: track 50.3 -> 53.4 mm
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
Commit message: Final v1 version
Parts:
- flipped L1 to the bottom, turned to 0 degrees
- flipped L2 to the bottom, turned to 0 degrees
- flipped U$7 to the bottom, turned to 270 degrees
- flipped U$9 to the bottom
Routing:
- net D5*: track 64.0 -> 75.7 mm
- net VCC: track 88.8 -> 93.8 mm
Changed lines of the file:
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@@
 <grid distance="25" unitdist="mil" unit="mil" style="lines" multiple="1" display="yes" altdistance="3.25" altunitdist="mil" altunit="mil"/>
 <layers>
-<layer number="1" name="Top" color="4" fill="1" visible="no" active="yes"/>
-<layer number="16" name="Bottom" color="1" fill="1" visible="no" active="yes"/>
+<layer number="1" name="Top" color="4" fill="1" visible="yes" active="yes"/>
+<layer number="16" name="Bottom" color="1" fill="1" visible="yes" active="yes"/>
 <layer number="17" name="Pads" color="2" fill="1" visible="yes" active="yes"/>
 <layer number="18" name="Vias" color="2" fill="1" visible="yes" active="yes"/>
@@
 <attribute name="VALUE" x="62.87135" y="26.95575" size="1.27" layer="28" rot="MR270"/>
 </element>
-<element name="U$9" library="lpatiny" package="LED-TRICOLOR-THROUGHHOLE" value="RGB-COMMON-CATHODE" x="64.77" y="12.065" rot="R270"/>
+<element name="U$9" library="lpatiny" package="LED-TRICOLOR-THROUGHHOLE" value="RGB-COMMON-CATHODE" x="64.77" y="12.065" rot="MR270"/>
 <element name="R7" library="rcl" package="R0805" value="1k" x="53.975" y="48.5648" rot="MR180"/>
 <element name="BKLD1" library="adafruit" package="CHIP-LED0805" value="RED" x="53.975" y="46.355" rot="MR270"/>
@@
 <attribute name="VALUE" x="52.07" y="27.305" size="1.27" layer="28" rot="MR0"/>
 </element>
-<element name="L1" library="SparkFun" package="LED5MM" value="UV" x="43.815" y="27.94" rot="R180"/>
-<element name="U$7" library="lpatiny" package="TSL237" value="TSL237" x="17.78" y="12.065" rot="R90"/>
+<element name="L1" library="SparkFun" package="LED5MM" value="UV" x="43.815" y="27.94" rot="MR0"/>
+<element name="U$7" library="lpatiny" package="TSL237" value="TSL237" x="17.78" y="12.065" rot="MR270"/>
 <element name="U$12" library="lpatiny" package="JST-2-XH" value="CONN2" x="63.5" y="68.58" rot="MR90"/>
 <element name="D7" library="lpatiny" package="LED-1206" value="1N581D1206" x="80.01" y="62.23" smashed="yes" rot="MR90">
@@
 <attribute name="VALUE" x="52.07" y="20.955" size="1.27" layer="28" rot="MR0"/>
 </element>
-<element name="L2" library="led" package="LED3MM" value="UV" x="43.815" y="24.765" rot="R180"/>
+<element name="L2" library="led" package="LED3MM" value="UV" x="43.815" y="24.765" rot="MR0"/>
 <element name="CON_ISP1" library="lpatiny" package="TINYISP" value="SPI" x="5.715" y="50.8" rot="MR90">
 <attribute name="MF" value="" x="5.715" y="50.8" size="1.778" layer="28" rot="MR90" display="off"/>
@@
 <via x="37.0459" y="54.8005" extent="1-16" drill="0.3048" shape="square"/>
 <wire x1="37.0459" y1="54.8005" x2="19.05" y2="54.8005" width="0.4064" layer="1"/>
-<wire x1="19.05" y1="54.8005" x2="19.05" y2="14.097" width="0.4064" layer="1"/>
-<wire x1="19.05" y1="14.097" x2="20.32" y2="14.097" width="0.4064" layer="1"/>
+<wire x1="19.05" y1="54.8005" x2="19.05" y2="20.447" width="0.4064" layer="1"/>
+<wire x1="19.05" y1="20.447" x2="24.13" y2="20.447" width="0.4064" layer="1"/>
+<wire x1="24.13" y1="20.447" x2="24.13" y2="10.033" width="0.4064" layer="1"/>
+<wire x1="24.13" y1="10.033" x2="20.32" y2="10.033" width="0.4064" layer="1"/>
 </signal>
 <signal name="VUSB">
@@
 <wire x1="36.2204" y1="54.7751" x2="36.2204" y2="53.975" width="0.4064" layer="16"/>
 <wire x1="36.2204" y1="53.975" x2="40.8051" y2="53.975" width="0.4064" layer="16"/>
-<wire x1="20.32" y1="12.065" x2="17.78" y2="12.065" width="0.4064" layer="1"/>
-<wire x1="17.78" y1="12.065" x2="17.78" y2="44.765" width="0.4064" layer="1"/>
+<wire x1="17.78" y1="18.415" x2="17.78" y2="44.765" width="0.4064" layer="1"/>
 <wire x1="17.78" y1="44.765" x2="24.13" y2="44.765" width="0.4064" layer="16"/>
 <via x="17.78" y="44.765" extent="1-16" drill="0.3048" shape="square"/>
+<wire x1="17.78" y1="18.415" x2="22.86" y2="18.415" width="0.4064" layer="1"/>
+<wire x1="22.86" y1="18.415" x2="22.86" y2="12.065" width="0.4064" layer="1"/>
+<wire x1="22.86" y1="12.065" x2="20.32" y2="12.065" width="0.4064" layer="1"/>
 <wire x1="46.225" y1="44.45" x2="62.4586" y2="45.1612" width="0" layer="19" extent="16-16"/>
 <wire x1="31.03" y1="48.4" x2="33.655" y2="54.7751" width="0" layer="19" extent="16-16"/>
