File: fridge/fridge.brd (EAGLE design)
At the start: 99.1 x 73.7 mm, 54 parts, among them IC1 MCP1703-33, IC2 MCP1703-50, J2 RJ12RIGHTANGLE-I2C, Q1 DMP1045U, U1 MCP73831T, X2 8MHz, X4 MINI-USB

Commit message: work on v1.0.1
Parts:
- removed C3: 10µF, microbuilder:0805
- removed D5: 1N581D1206, lpatiny:LED-1206
- removed L1: UV, SparkFun:LED5MM
- removed L2: UV, led:LED3MM
- removed LED1: RED, microbuilder:CHIPLED_0805
- removed LED2: GREEN, microbuilder:CHIPLED_0805
- removed Q1: DMP1045U, dp_devices:SOT-23
- removed R1, R4: 470, microbuilder:0805
- removed R2, R9: 1k, rcl:R0805
- removed R3: 100k, microbuilder:0805
- removed R5: 10K\, microbuilder:0805
- removed RL2, RL4: 150, rcl:R0805
- removed RL3: 100, rcl:R0805
- removed U$12: CONN2, lpatiny:JST-2-XH
- removed U$7: TSL237, lpatiny:TSL237
- removed U$9: RGB-COMMON-CATHODE, lpatiny:LED-TRICOLOR-THROUGHHOLE
- removed U1: MCP73831T, microbuilder:SOT23-5
- IC1: value MCP1703-33 -> MCP1703-50
- moved RK7 1.27 mm to (46.4, 56.5)
- moved D4 0.63 mm to (83.8, 62.2)
Connections:
- removed net N$10: RL3.1, U$9.BLU
- removed net N$13: RL2.1, U$9.RED
- removed net N$15: C2.1, D4.C, D5.A, D7.C, D8.C, IC2.3, LED1.A, Q1.1, R3.2, U1.4
- removed net N$3: L1.A, R9.2
- removed net N$4: LED1.C, R1.1
- removed net N$5: R1.2, R4.2, U1.1
- removed net N$6: R5.1, U1.5
- removed net N$7: LED2.A, R4.1
- removed net N$8: L2.A, R2.2
- removed net N$9: RL4.2, U$9.GRN
- removed net VBAT1: C3.1, Q1.3, U$12.2, U1.3
- new net N$19: C2.1, D4.C, D7.C, D8.C, IC2.3
- net A0: no longer RL2.2
- net A1: no longer RL4.1
- net A2: no longer RL3.2
- net A3: no longer R2.1
- net A4: no longer R9.1
- net D5*: no longer U$7.OUT
- net GND: no longer C3.2, L1.K, L2.K, LED2.C, R3.1, R5.2, U$12.1, U$7.GND, U$9.GND, U1.2
- net VCC: no longer U$7.VDD
- net VDD: no longer D5.C, Q1.2
Routing:
- net VCC: track 308.5 -> 86.2 mm, vias 2 -> 1
- net N$15: track 69.1 -> 0.00 mm
- net VBAT1: track 57.7 -> 0.00 mm
- net N$19: track 0.00 -> 52.8 mm
- net GND: track 153.1 -> 117.6 mm, vias 11 -> 9
- net N$5: track 15.2 -> 0.00 mm
- net N$10: track 15.2 -> 0.00 mm
- net D5*: track 75.7 -> 62.7 mm
- net N$9: track 11.2 -> 0.00 mm
- net N$3: track 7.30 -> 0.00 mm
- net N$8: track 6.67 -> 0.00 mm
- net N$13: track 5.83 -> 0.00 mm
- net A3: track 47.3 -> 42.2 mm
- net VDD: track 13.4 -> 8.88 mm
- net A4: track 42.0 -> 37.9 mm
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Other:
- board text removed: "Simple spectrophotometer V 1.0.1"
